File: Music32v3/Music32v3.kicad_pcb (KiCad board)
At the start: 4 copper layers, 46 x 100 mm, 16 parts, among them J1 USB_C_Receptacle_USB2.0, J2 Micro_SD_Card_Det1, J3 PJ-316A-6A, SW1 Vol+, SW2 Select, SW3 Vol-, SW4 PP, SW5 RW, SW6 FF, SW7 HOME, SW9 Power, U1 ST7889 2" LCD, U3 Sk-3393, U4 SRGP400200, U5 ESP32-WROOM-32E__16MB_

Commit message: pcb done
Parts:
- added BT1: Battery_Cell, Music:HCZZ0001-2, F.Cu at (111.8, 137.7)
- added C1: 1uF, Capacitor_SMD:C_0402_1005Metric, F.Cu at (126.4, 90.3)
- added C10: 1uF, Capacitor_SMD:C_0402_1005Metric, F.Cu at (115.2, 143.7)
- added C11: 4.7uF, Capacitor_SMD:C_0402_1005Metric, F.Cu at (117.7, 132.2)
- added C12: 22uf, Capacitor_SMD:C_0805_2012Metric, F.Cu at (129.0, 76.8)
- added C13: 1uF, Capacitor_SMD:C_0402_1005Metric, F.Cu at (120.3, 141.5)
- added C14: 22uf, Capacitor_SMD:C_0805_2012Metric, F.Cu at (131.9, 74.0)
- added C15: 22uf, Capacitor_SMD:C_0805_2012Metric, F.Cu at (144.7, 96.8)
- added C16: 22uf, Capacitor_SMD:C_0805_2012Metric, F.Cu at (118.2, 126.7)
- added C17: 1uF, Capacitor_SMD:C_0402_1005Metric, F.Cu at (123.6, 146.6)
- added C18: 1uF, Capacitor_SMD:C_0402_1005Metric, F.Cu at (119.1, 144.8)
- added C19: 24pF, Capacitor_SMD:C_0402_1005Metric, F.Cu at (144.6, 147.7)
- added C2: 0.1uF, Capacitor_SMD:C_0402_1005Metric, F.Cu at (131.5, 118.8)
- added C20: 24pF, Capacitor_SMD:C_0402_1005Metric, F.Cu at (144.5, 142.3)
- added C21: 1uF, Capacitor_SMD:C_0402_1005Metric, F.Cu at (136.0, 146.2)
- added C22: 1uF, Capacitor_SMD:C_0402_1005Metric, F.Cu at (131.7, 131.5)
- added C23: 1uF, Capacitor_SMD:C_0402_1005Metric, F.Cu at (143.8, 131.6)
- added C24: 1uF, Capacitor_SMD:C_0402_1005Metric, F.Cu at (140.1, 147.2)
- added C25: 1uF, Capacitor_SMD:C_0402_1005Metric, F.Cu at (141.9, 146.3)
- added C26: 1uF, Capacitor_SMD:C_0402_1005Metric, F.Cu at (143.8, 126.1)
- added C27: 1uF, Capacitor_SMD:C_0402_1005Metric, F.Cu at (131.7, 126.1)
- added C28: 4.7uF, Capacitor_SMD:C_0402_1005Metric, F.Cu at (136.1, 140.0)
- added C29: 4.7uF, Capacitor_SMD:C_0402_1005Metric, F.Cu at (134.2, 139.1)
- added C3: 1uF, Capacitor_SMD:C_0402_1005Metric, F.Cu at (138.0, 93.2)
- added C30: 1uF, Capacitor_SMD:C_0402_1005Metric, F.Cu at (143.8, 128.8)
- added C31: 1uF, Capacitor_SMD:C_0402_1005Metric, F.Cu at (131.7, 128.8)
- added C32: 4.7uF, Capacitor_SMD:C_0402_1005Metric, F.Cu at (138.0, 140.0)
- added C33: 1uF, Capacitor_SMD:C_0402_1005Metric, F.Cu at (108.2, 98.7)
- added C34: 0.1uF, Capacitor_SMD:C_0402_1005Metric, F.Cu at (151.2, 135.0)
- added C35: 0.1uF, Capacitor_SMD:C_0402_1005Metric, F.Cu at (151.2, 137.5)
- added C36: 1uF, Capacitor_SMD:C_0402_1005Metric, F.Cu at (131.3, 67.8)
- added C37: 1uF, Capacitor_SMD:C_0402_1005Metric, F.Cu at (131.3, 68.7)
- added C38: 1uF, Capacitor_SMD:C_0402_1005Metric, F.Cu at (139.5, 67.7)
- added C39: 1uF, Capacitor_SMD:C_0402_1005Metric, F.Cu at (139.5, 69.5)
- added C4: 0.1uF, Capacitor_SMD:C_0402_1005Metric, F.Cu at (140.7, 96.4)
- added C40: 1uF, Capacitor_SMD:C_0402_1005Metric, F.Cu at (139.5, 66.8)
- added C41: 1uF, Capacitor_SMD:C_0402_1005Metric, F.Cu at (139.5, 68.6)
- added C42: 22uf, Capacitor_SMD:C_0805_2012Metric, F.Cu at (133.8, 73.9)
- added C43: 1uF, Capacitor_SMD:C_0402_1005Metric, F.Cu at (136.0, 73.0)
- added C44: 1uF, Capacitor_SMD:C_0402_1005Metric, F.Cu at (134.9, 64.9)
- added C45: 1uF, Capacitor_SMD:C_0402_1005Metric, F.Cu at (135.8, 64.9)
- added C46: 1uF, Capacitor_SMD:C_0402_1005Metric, F.Cu at (136.7, 64.9)
- added C47: 1uF, Capacitor_SMD:C_0402_1005Metric, F.Cu at (137.6, 64.9)
- added C48: 1uF, Capacitor_SMD:C_0402_1005Metric, F.Cu at (137.7, 72.6)
- added C49: 47nF, Capacitor_SMD:C_0402_1005Metric, F.Cu at (131.4, 71.3)
- added C5: 0.1uf, Capacitor_SMD:C_0402_1005Metric, F.Cu at (141.6, 96.4)
- added C50: 4.7uF, Capacitor_SMD:C_0402_1005Metric, F.Cu at (142.0, 51.8)
- added C6: 22uf, Capacitor_SMD:C_0805_2012Metric, F.Cu at (144.7, 94.8)
- added C7: 22uf, Capacitor_SMD:C_0805_2012Metric, F.Cu at (144.7, 92.8)
- added C8: 1uF, Capacitor_SMD:C_0402_1005Metric, F.Cu at (123.5, 139.0)
- added C9: 0.1uF, Capacitor_SMD:C_0402_1005Metric, F.Cu at (117.5, 136.9)
- added D1: DSS34, Diode_SMD:D_SOD-123F, F.Cu at (120.8, 134.3)
- added D2: LED_Small, LED_SMD:LED_0603_1608Metric, F.Cu at (121.0, 148.2)
- added D3: LED_Small, LED_SMD:LED_0603_1608Metric, F.Cu at (119.4, 148.2)
- added D4: LED, LED_SMD:LED_0603_1608Metric, F.Cu at (141.0, 148.8)
- added F1: Polyfuse, Fuse:Fuse_0603_1608Metric, F.Cu at (126.3, 140.4)
- added F2: Polyfuse, Fuse:Fuse_0603_1608Metric, F.Cu at (116.0, 145.3)
- added FB1: 100ohm@100MHz, Resistor_SMD:R_0402_1005Metric, F.Cu at (134.2, 137.1)
- added Q1: CJ3134K KF, Package_TO_SOT_SMD:SOT-723, F.Cu at (122.4, 91.9)
- added Q2: CJ3134K KF, Package_TO_SOT_SMD:SOT-723, F.Cu at (115.2, 142.1)
- added Q3: CJ3134K KF, Package_TO_SOT_SMD:SOT-723, F.Cu at (117.5, 138.5)
- added Q4: YJQD30P02A, Music:YJQD30P02A_DFN3.3x3.3, F.Cu at (120.6, 137.5)
- added Q5: CJ3139K, Package_TO_SOT_SMD:SOT-723, F.Cu at (111.1, 97.9)
- added Q6: CJ3134K KF, Package_TO_SOT_SMD:SOT-723, F.Cu at (146.5, 140.7)
- added Q7: CJ3134K KF, Package_TO_SOT_SMD:SOT-723, F.Cu at (148.6, 140.7)
- added R1: 10K, Resistor_SMD:R_0402_1005Metric, F.Cu at (117.5, 74.1)
- added R10: 220, Resistor_SMD:R_0402_1005Metric, F.Cu at (118.6, 122.9)
- added R11: 10K, Resistor_SMD:R_0402_1005Metric, F.Cu at (132.5, 118.8)
- added R12: 1M, Resistor_SMD:R_0402_1005Metric, F.Cu at (139.4, 90.6)
- added R13: 5.1K, Resistor_SMD:R_0402_1005Metric, F.Cu at (142.4, 74.8)
- added R14: 10K, Resistor_SMD:R_0402_1005Metric, F.Cu at (139.7, 96.4)
- added R15: 10k, Resistor_SMD:R_0402_1005Metric, F.Cu at (142.5, 96.4)
- added R16: 2K, Resistor_SMD:R_0402_1005Metric, F.Cu at (132.1, 64.9)
- added R17: 2K, Resistor_SMD:R_0402_1005Metric, F.Cu at (133.0, 64.9)
- added R18: 1M, Resistor_SMD:R_0402_1005Metric, F.Cu at (142.6, 123.0)
- added R19: 1M, Resistor_SMD:R_0402_1005Metric, F.Cu at (123.5, 137.9)
- added R2: 10K, Resistor_SMD:R_0402_1005Metric, F.Cu at (117.5, 75.1)
- added R20: 1M, Resistor_SMD:R_0402_1005Metric, F.Cu at (117.5, 135.9)
- added R21: 5.1K, Resistor_SMD:R_0402_1005Metric, F.Cu at (128.5, 141.3)
- added R22: 5.1K, Resistor_SMD:R_0402_1005Metric, F.Cu at (131.9, 141.3)
- added R23: 1M, Resistor_SMD:R_0402_1005Metric, F.Cu at (123.5, 136.6)
- added R24: 2K, Resistor_SMD:R_0402_1005Metric, F.Cu at (122.9, 148.2)
- added R25: 2K, Resistor_SMD:R_0402_1005Metric, F.Cu at (117.4, 148.1)
- added R26: 2K, Resistor_SMD:R_0402_1005Metric, F.Cu at (122.4, 142.1)
- added R27: 100K, Resistor_SMD:R_0402_1005Metric, F.Cu at (133.7, 123.1)
- added R28: DNP, Resistor_SMD:R_0402_1005Metric, F.Cu at (141.7, 123.0)
- added R29: 2K, Resistor_SMD:R_0402_1005Metric, F.Cu at (138.4, 148.8)
- added R3: 1M, Resistor_SMD:R_0402_1005Metric, F.Cu at (122.4, 93.3)
- added R30: DNP, Resistor_SMD:R_0402_1005Metric, F.Cu at (134.7, 123.1)
- added R31: DNP, Resistor_SMD:R_0402_1005Metric, F.Cu at (135.6, 118.5)
- added R32: 1M, Resistor_SMD:R_0402_1005Metric, F.Cu at (112.7, 97.9)
- added R33: DNP, Resistor_SMD:R_0402_1005Metric, F.Cu at (146.5, 139.1)
- added R34: 4K7, Resistor_SMD:R_0402_1005Metric, F.Cu at (148.6, 139.1)
- added R35: 10K, Resistor_SMD:R_0402_1005Metric, F.Cu at (133.9, 64.9)
- added R36: 0R, Resistor_SMD:R_0402_1005Metric, F.Cu at (138.2, 75.0)
- added R37: 10K, Resistor_SMD:R_0402_1005Metric, F.Cu at (138.7, 96.4)
- added R38: 220R, Resistor_SMD:R_0402_1005Metric, F.Cu at (130.1, 64.9)
- added R39: 220R, Resistor_SMD:R_0402_1005Metric, F.Cu at (140.1, 51.8)
- added R4: 10R, Resistor_SMD:R_0402_1005Metric, F.Cu at (125.0, 92.7)
- added R40: 1M, Resistor_SMD:R_0402_1005Metric, F.Cu at (131.1, 64.9)
- added R41: 10K, Resistor_SMD:R_0402_1005Metric, F.Cu at (139.5, 71.5)
- added R42: 2K, Resistor_SMD:R_0402_1005Metric, F.Cu at (142.0, 52.7)
- added R43: 2K, Resistor_SMD:R_0402_1005Metric, F.Cu at (142.0, 54.7)
- added R44: 33R, Resistor_SMD:R_0402_1005Metric, F.Cu at (139.5, 72.5)
- added R45: 33R, Resistor_SMD:R_0402_1005Metric, F.Cu at (139.5, 70.5)
- added R5: 2K, Resistor_SMD:R_0402_1005Metric, F.Cu at (117.5, 88.1)
- added R6: 1K, Resistor_SMD:R_0402_1005Metric, F.Cu at (128.3, 136.4)
- added R7: 1K, Resistor_SMD:R_0402_1005Metric, F.Cu at (136.9, 124.9)
- added R8: 1M, Resistor_SMD:R_0402_1005Metric, F.Cu at (132.0, 90.4)
- added R9: 1K, Resistor_SMD:R_0402_1005Metric, F.Cu at (137.9, 124.9)
- added SW8: RESET, Music:TS3315A, F.Cu at (143.6, 86.7)
- added TP1: TestPoint, TestPoint:TestPoint_Pad_D2.0mm, F.Cu at (126.5, 129.6)
- added TP10: TestPoint, TestPoint:TestPoint_Pad_D2.0mm, F.Cu at (140.2, 83.4)
- added TP11: TestPoint, TestPoint:TestPoint_Pad_D2.0mm, F.Cu at (120.5, 57.1)
- added TP12: TestPoint, TestPoint:TestPoint_Pad_D2.0mm, F.Cu at (120.5, 61.0)
- added TP13: TestPoint, TestPoint:TestPoint_Loop_D2.50mm_Drill1.0mm, F.Cu at (117.7, 53.1)
- added TP14: TestPoint, TestPoint:TestPoint_Pad_D2.0mm, F.Cu at (115.8, 79.3)
- added TP15: TestPoint, TestPoint:TestPoint_Pad_D2.0mm, F.Cu at (114.9, 127.8)
- added TP16: TestPoint, TestPoint:TestPoint_Pad_D2.0mm, F.Cu at (126.1, 137.2)
- added TP17: TestPoint, TestPoint:TestPoint_Pad_D2.0mm, F.Cu at (121.5, 131.4)
- added TP18: TestPoint, TestPoint:TestPoint_Pad_D2.0mm, F.Cu at (136.0, 76.5)
- added TP19: TestPoint, TestPoint:TestPoint_Pad_D2.0mm, F.Cu at (112.2, 129.7)
- added TP2: TestPoint, TestPoint:TestPoint_Pad_D2.0mm, F.Cu at (122.5, 96.0)
- added TP20: TestPoint, TestPoint:TestPoint_Pad_D2.0mm, F.Cu at (115.6, 65.2)
- added TP21: TestPoint, TestPoint:TestPoint_Pad_D1.0mm, F.Cu at (119.0, 121.2)
- added TP22: TestPoint, TestPoint:TestPoint_Pad_D1.0mm, F.Cu at (121.0, 119.9)
- added TP23: TestPoint, TestPoint:TestPoint_Pad_D1.0mm, F.Cu at (127.8, 124.9)
- added TP24: TestPoint, TestPoint:TestPoint_Pad_D1.0mm, F.Cu at (125.2, 121.0)
- added TP25: TestPoint, TestPoint:TestPoint_Pad_D1.0mm, F.Cu at (124.7, 118.6)
- added TP26: TestPoint, TestPoint:TestPoint_Pad_D1.0mm, F.Cu at (121.3, 114.8)
- added TP27: TestPoint, TestPoint:TestPoint_Pad_D2.0mm, F.Cu at (118.1, 97.5)
- added TP28: TestPoint, TestPoint:TestPoint_Pad_D2.0mm, F.Cu at (109.0, 95.7)
- added TP29: TestPoint, TestPoint:TestPoint_Pad_D2.0mm, F.Cu at (151.4, 140.6)
- added TP3: TestPoint, TestPoint:TestPoint_Pad_D2.0mm, F.Cu at (125.4, 94.7)
- added TP30: TestPoint, TestPoint:TestPoint_Pad_D1.5mm, F.Cu at (124.5, 114.1)
- added TP31: TestPoint, TestPoint:TestPoint_Pad_D1.5mm, F.Cu at (144.8, 133.6)
- added TP32: TestPoint, TestPoint:TestPoint_Pad_D2.0mm, F.Cu at (120.7, 67.6)
- added TP33: TestPoint, TestPoint:TestPoint_Pad_D1.5mm, F.Cu at (126.4, 82.6)
- added TP34: TestPoint, TestPoint:TestPoint_Pad_D1.5mm, F.Cu at (124.2, 78.6)
- added TP35: TestPoint, TestPoint:TestPoint_Pad_D1.5mm, F.Cu at (125.4, 74.6)
- added TP36: TestPoint, TestPoint:TestPoint_Pad_D2.0mm, F.Cu at (133.9, 83.8)
- added TP4: TestPoint, TestPoint:TestPoint_Pad_D1.5mm, F.Cu at (130.9, 95.8)
- added TP6: TestPoint, TestPoint:TestPoint_Pad_D2.0mm, F.Cu at (127.0, 87.3)
- added TP7: TestPoint, TestPoint:TestPoint_Pad_D2.0mm, F.Cu at (121.8, 124.9)
- added TP8: TestPoint, TestPoint:TestPoint_Pad_D1.5mm, F.Cu at (139.4, 88.2)
- added TP9: TestPoint, TestPoint:TestPoint_Pad_D2.0mm, F.Cu at (139.0, 80.5)
- added U10: TP4057, Package_TO_SOT_SMD:SOT-23-6, F.Cu at (121.7, 144.3)
- added U11: SN74LVC1G3157, Package_TO_SOT_SMD:SOT-363_SC-70-6, F.Cu at (133.8, 131.1)
- added U12: SN74LVC1G3157, Package_TO_SOT_SMD:SOT-363_SC-70-6, F.Cu at (141.7, 131.1)
- added U13: ~, Music:SL2.1S, F.Cu at (138.9, 144.2)
- added U14: SN74LVC1G3157, Package_TO_SOT_SMD:SOT-363_SC-70-6, F.Cu at (133.8, 128.3)
- added U15: SN74LVC1G3157, Package_TO_SOT_SMD:SOT-363_SC-70-6, F.Cu at (141.7, 128.3)
- added U16: GL823, Package_SO:SSOP-16_3.9x4.9mm_P0.635mm, F.Cu at (137.5, 136.0)
- added U17: SN74LVC1G3157, Package_TO_SOT_SMD:SOT-363_SC-70-6, F.Cu at (133.8, 125.6)
- added U18: SN74LVC1G3157, Package_TO_SOT_SMD:SOT-363_SC-70-6, F.Cu at (141.7, 125.6)
- added U19: TPD2EUSB30, Package_TO_SOT_SMD:Texas_DRT-3, F.Cu at (112.4, 115.0)
- added U2: MAX17048, Package_DFN_QFN:DFN-8-1EP_2x2mm_P0.5mm_EP0.8x1.6mm, F.Cu at (137.7, 91.1)
- added U20: CH340X, Package_SO:MSOP-10_3x3mm_P0.5mm, F.Cu at (147.5, 136.5)
- added U21: TPD2EUSB30, Package_TO_SOT_SMD:Texas_DRT-3, F.Cu at (118.0, 115.0)
- added U22: TPD2EUSB30, Package_TO_SOT_SMD:Texas_DRT-3, F.Cu at (115.2, 115.0)
- added U23: ES8327, Package_DFN_QFN:QFN-32-1EP_4x4mm_P0.4mm_EP2.9x2.9mm_ThermalVias, F.Cu at (135.2, 69.2)
- added U6: TPD2EUSB30, Package_TO_SOT_SMD:Texas_DRT-3, F.Cu at (130.2, 141.5)
- added U7: SSP6206-18NR, Package_TO_SOT_SMD:SOT-23, F.Cu at (129.0, 73.9)
- added U8: XC6210B332MR, Package_TO_SOT_SMD:SOT-23-5, F.Cu at (118.2, 129.7)
- added U9: SSP61CC3602MR, Package_TO_SOT_SMD:SOT-23-3, F.Cu at (118.0, 141.7)
- added Y1: 12MHz, Crystal:Crystal_SMD_3225-4Pin_3.2x2.5mm, F.Cu at (144.6, 145.0)
- moved U5 1.30 mm to (137.3, 107.6)
Routing:
- net +3V3: track 0.00 -> 346.9 mm, vias 0 -> 12
- net GND: track 0.00 -> 143.2 mm, vias 16 -> 159
- net BATT+: track 0.00 -> 122.0 mm, vias 0 -> 6
- net BUTTONS: track 0.00 -> 117.0 mm, vias 0 -> 6
- net MCLK_TXD: track 0.00 -> 83.2 mm, vias 0 -> 2
- net SCL: track 0.00 -> 67.7 mm, vias 0 -> 4
- net EN: track 0.00 -> 66.7 mm, vias 0 -> 4
- net DAT1_SD: track 0.00 -> 63.5 mm, vias 0 -> 4
- net SDA: track 0.00 -> 58.7 mm, vias 0 -> 3
- net VBUS: track 0.00 -> 52.9 mm, vias 0 -> 2
- net MOSI_UC: track 0.00 -> 52.8 mm, vias 0 -> 2
- net CLK_SD: track 0.00 -> 52.5 mm, vias 0 -> 4
- net DAT0/MISO_SD: track 0.00 -> 51.7 mm, vias 0 -> 4
- net SCLK: track 0.00 -> 49.8 mm
- net SD_SELECT: track 0.00 -> 48.2 mm, vias 0 -> 6
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- added copper zone on In1.Cu, net GND
- added copper zone on In2.Cu, net GND
- added copper zone on F.Cu, net Net-(Q4A-D2-Pad7)
Other:
- board text added: "+-"
- board text added: "1V8"
- board text added: "3V3"
- board text added: "5V"
- board text added: "BL_EN"
- board text added: "BUTTONS"
- board text added: "Batt+"
- board text added: "DSPLY_CS"
- board text added: "DSPLY_DC"
- board text added: "DSPLY_RST"
- board text added: "DVDD"
- board text added: "EN"
- board text added: "FF"
- board text added: "FUEL_INT"
- board text added: "GND"
- board text added: "HOLD"
- board text added: "HOME"
- board text added: "HSET INT"
- board text added: "IO0"
- board text added: "LRCK"
- board text added: "MCK TXD"
- board text added: "OFF"
- board text added: "ON"
- board text added: "PP"
- board text added: "PWR"
- board text added: "PWR/HLD"
- board text added: "RST"
- board text added: "RW"
- board text added: "SCL"
- board text added: "SCLK"
- board text added: "SDA"
- board text added: "SDIN"
- board text added: "SDOUT"
- board text added: "SDPWR"
- board text added: "SD_DET"
- board text added: "SD_VDD"
- board text added: "VIN"
- board text added: "VOL+"
- board text added: "VOL-"

Commit message: Update
Routing:
- net D+: track 16.1 -> 17.2 mm
- net UART_D-: track 11.5 -> 12.2 mm
- net UART_D+: track 11.5 -> 12.2 mm

Commit message: pdf schematic
Parts:
- added TP5: TestPoint, TestPoint:TestPoint_Pad_D2.0mm, F.Cu at (122.7, 84.5)
- C5: value 0.1uf -> 0.1uF
- R15: value 10k -> 10K
- R27: value 100K -> 1M
- TP8: footprint TestPoint:TestPoint_Pad_D1.5mm -> TestPoint:TestPoint_Pad_D2.0mm
Routing:
- net CLK_UC: track 45.4 -> 60.2 mm, vias 1 -> 2
- net +3V3: track 346.9 -> 345.3 mm, vias 12 -> 13
Other:
- board text added: "DSPLY_CLK"
